Commit message: urdf section

File: Part_2/minimal_robot_description/minimal_robot_description_wo_collision.urdf (robot description, URDF)
Before this commit: robot one_DOF_robot, 3 links, 2 joints
Links:
- link link1: geometry visual box size=0.2 0.2 1
- link link2: geometry visual cylinder length=1 radius=0.1
