Commit message: work in ptIII

File: Part_3/simple_camera_model/simple_camera_model.xacro (robot description, xacro)
@@ -4,14 +4,6 @@
       <origin xyz="0.0 0.0 0.0"/>
   </link>
-  <joint name="world_joint" type="fixed">
+  <joint name="camera_joint" type="fixed">
       <parent link="world"/>
-      <child link="camera_stand"/>
-      <origin rpy="0.0 0.0 0.0" xyz="0.0 0.0 0.0"/>
-  </joint>
-  <link name="camera_stand">
-    <origin rpy="0.0 0.0 0.0" xyz="0.0 0.0 0.5"/>
-  </link>
-  <joint name="camera_joint" type="fixed">
-      <parent link="camera_stand"/>
       <child link="camera_link"/>
       <origin rpy="0.0 1.5708 1.5708" xyz="0 0.0 0.5"/>
@@ -23,5 +15,4 @@
         <box size="0.03 0.01 0.01"/>
       </geometry>
-      <material name="red"/>
     </visual>
     <inertial>
@@ -30,5 +21,4 @@
       <inertia ixx="1e-6" ixy="0" ixz="0" iyy="1e-6" iyz="0" izz="1e-6" />
     </inertial>
-  <!--origin rpy="0.0 0.0 0.0" xyz="0.0 0.2 0.8"/-->
   </link>
   <!-- camera simulator plug-in -->
@@ -49,7 +39,4 @@
         <noise>
           <type>gaussian</type>
-          <!-- Noise is sampled independently per pixel on each frame.
-               That pixel's noise value is added to each of its color
-               channels, which at that point lie in the range [0,1]. -->
           <mean>0.0</mean>
           <stddev>0.000</stddev>
@@ -63,5 +50,4 @@
         <cameraInfoTopicName>camera_info</cameraInfoTopicName>
         <frameName>camera_link</frameName>
-        <!--hackBaseline>0.07</hackBaseline-->
         <distortionK1>0.0</distortionK1>
         <distortionK2>0.0</distortionK2>
