Commit message: part3 stuff

File: Part_3/simple_camera_model/multi_camera_model.xacro (robot description, xacro)
@@ -43,4 +43,11 @@
   <link name="left_camera_optical_frame_mid">
   </link>
+    <link name="left_camera_ref_frame">
+  </link>
+  <joint name="left_camera_ref_joint" type="fixed">
+      <parent link="left_camera_body"/>
+      <child link="left_camera_ref_frame"/>
+      <origin rpy="-1.5708 0 0" xyz="0 0 0"/>
+  </joint>
   <joint name="left_camera_optical_joint" type="fixed">
       <parent link="left_camera_optical_frame_mid"/>
@@ -60,5 +67,5 @@
   </joint>
 <!-- start of stereo camera plug-in -->
-  <gazebo reference="left_camera_body">
+  <gazebo reference="left_camera_ref_frame">
   <!--gazebo reference="left_camera_optical_frame"-->
     <sensor type="multicamera" name="stereo_camera">
@@ -82,5 +89,5 @@
       </camera>
       <camera name="right">
-        <pose>0.02 0 0 0 0 0</pose>
+        <pose>0 -0.02  0 0 0 0</pose>
         <horizontal_fov>0.6</horizontal_fov>
         <image>
