Commit message: part-6 edits

File: Part_3/simple_camera_model/simple_kinect_model3.xacro (robot description, xacro)
@@ -2,4 +2,20 @@
 <robot xmlns:xacro="http://www.ros.org/wiki/xacro" name="kinect_link">
  <!-- ADD a Kinect sensor: first the visual/collision/inertial box -->
+  <link name="world">
+      <origin xyz="0.0 0.0 0.0"/>
+  </link>
+    <link name="base_link">
+  </link>
+  <joint name="kinect_jnt" type="fixed">
+      <parent link="base_link"/>
+      <child link="kinect_link"/>
+      <!--origin rpy="0.0 1.5708 1.5708" xyz="0 0.0 0.5"/-->
+      <axis xyz="0 1 0" />
+      <origin xyz="0.027 0.0 1.810" rpy="0.0 1.2 0"/>
+  </joint>
+    <joint name="world_jnt" type="fixed">
+      <parent link="world"/>
+      <child link="base_link"/>
+  </joint>
     <link name="kinect_link">
       <collision>
@@ -27,11 +43,12 @@
   <!--the above displays a box meant to imply Kinect-->
   <!--now set the position/orientation of the above box: -->
-  <joint name="kinect_joint" type="fixed">
+  <!--joint name="kinect_joint" type="fixed">
       <axis xyz="0 1 0" />
-      <origin xyz="0.2 0.0 0.9" rpy="0.0 1.2 0"/>
-      <parent link="torso"/>
+      <origin xyz="0.2 0.0 1.9" rpy="0.0 1.2 0"/>
+      <parent link="kinect_stand"/>
       <child link="kinect_link"/>
-  </joint>
-  <!--  add kinect sensor emulation -->
+  </joint-->
+<!-- end wsn adding kinect link; -->
+  <!-- wsn: add kinect sensor emulation -->
 <gazebo reference="kinect_link">
     <sensor type="depth" name="openni_camera_camera">

File: Part_6/baxter_variations/baxter_on_pedestal.xacro (robot description, xacro)
@@ -2,14 +2,12 @@
 <robot
   xmlns:xacro="http://www.ros.org/wiki/xacro" name="baxter_on_pedestal">
-  <!--xacro:include filename="$(find baxter_on_mobot)/mobot_base.xacro" /-->
-  <!--xacro:include filename="$(find baxter_on_mobot)/baxter_base.urdf.xacro">
-    <xacro:arg name="gazebo" value="${gazebo}"/>
-  </xacro:include-->
-    <!-- Baxter Base URDF -->
+  <!-- Baxter Base URDF -->
   <xacro:include filename="$(find baxter_description)/urdf/baxter_base/baxter_base.urdf.xacro">
     <xacro:arg name="gazebo" value="${gazebo}"/>
   </xacro:include>
+  <!--grippers-->
   <xacro:include filename="$(find baxter_description)/urdf/left_end_effector.urdf.xacro" />
   <xacro:include filename="$(find baxter_description)/urdf/right_end_effector.urdf.xacro" />
+  <!--retrofit with Kinect and pedestal-->
   <xacro:include filename="$(find baxter_variations)/kinect_link.urdf.xacro" />
   <xacro:include filename="$(find baxter_variations)/baxter_pedestal.xacro" />
@@ -27,16 +25,3 @@
     <origin rpy="0 0 0 " xyz="0 0 0"/>
   </joint>
-  <!-- attach baxter torso to the mobile robot -->
-  <!--joint name="baxter_base_joint" type="fixed">
-    <parent link="mobot_top" />
-    <child link="base" />
-    <origin rpy="0 0 0 " xyz="0.1 0 0.06"/>
-  </joint-->
-  <!-- attach the kinect to the mobile robot
-  <joint name="kinect_joint" type="fixed">
-    <parent link="base_link" />
-    <child link="kinect_link" />
-    <origin rpy="0 0 0 " xyz="0.1 0 0.72"/>
-  </joint-->
-  <!-- kinect depth frame has a different viewpoint; publish it separately-->
 </robot>

File: Part_6/baxter_variations/baxter_pedestal.xacro (robot description, xacro)
@@ -2,10 +2,10 @@
 <robot
      xmlns:xacro="http://www.ros.org/wiki/xacro" name="pedestal">
-     <!-- define the base-link origin to lie at floor level, between the drive wheels-->
-     <!--main body is a simple box; origin is a center of box-->
+     <!-- a simple box onto which Baxter robot can be mounted-->
     <xacro:property name="bodylen" value="0.3" />
     <xacro:property name="bodywidth" value="0.3" />
     <xacro:property name="bodyheight" value="0.85" />
-    <!--link name="baxter_pedestal"-->
+    <!--this will be referred to as the "base_link", so code can be
+    compatible with baxter on mobot-->
     <link name="base_link">
         <visual>
