Commit message: removed comment

File: Part_6/baxter_variations/baxter_on_mobot.xacro (robot description, xacro)
@@ -15,10 +15,3 @@
     <origin rpy="0 0 0 " xyz="0.1 0 0.06"/>
   </joint>
-  <!-- attach the kinect to the mobile robot
-  <joint name="kinect_joint" type="fixed">
-    <parent link="base_link" />
-    <child link="kinect_link" />
-    <origin rpy="0 0 0 " xyz="0.1 0 0.72"/>
-  </joint-->
-  <!-- kinect depth frame has a different viewpoint; publish it separately-->
 </robot>
