Commit message: working on ur10 w/ vacuum gripper

File: Part_5/ur10_robot/ur10_launch/ur10_on_pedestal_w_sticky_fingers.xacro (robot description, xacro)
@@ -24,11 +24,54 @@
     <origin rpy="0 0 0 " xyz="0 0 0"/>
   </joint>
-  <gazebo>
-  <sensor name='virtual_vacuum_gripper' type='contact'>
-    <plugin name="virtual_vacuum_gripper" filename="libsticky_fingers.so">
+  <link name= "virtual_vacuum_gripper">
+       <visual>
+      <geometry>
+         <cylinder length="0.02" radius="0.04"/>
+      </geometry>
+      <material name="blue">
+        <color rgba="0 0 .8 1"/>
+      </material>
+    </visual>
+    <collision name="virtual_vacuum_gripper_collision">
+      <origin rpy="0 0 0" xyz = "0 0 0"/>
+      <geometry>
+          <box size= "0.02 0.02 0.04"/>
+        <!--cylinder length="0.02" radius="0.04"/-->
+      </geometry>
+      <surface>
+          <friction>
+              <ode>
+                  <mu>30.0</mu>
+                  <mu2>30.0</mu2>
+              </ode>
+          </friction>
+          <contact>
+              <ode>
+                  <kp>100000.0</kp>
+                  <kd>100.0</kd>
+                  <max_vel>1.0</max_vel>
+                  <min_depth>0.001</min_depth>
+              </ode>
+          </contact>
+      </surface>
+    </collision>
+    <inertial>
+        <mass value = "0.05"/>
+        <inertia ixx = "0.01" iyy="0.01" izz="0.01" ixy="0.0" ixz="0.0" iyz="0.0" />
+    </inertial>
+  </link>
+  <joint name="gripper_joint" type="fixed">
+    <parent link="tool0" />
+    <!--ur10 base link is child-->
+    <child link="virtual_vacuum_gripper" />
+    <origin rpy="0 0 0 " xyz="0 0 0.0"/>
+  </joint>
+  <gazebo reference= "virtual_vacuum_gripper">
+  <sensor name="virtual_vacuum_gripper_sticky" type="contact">
+    <plugin name="virtual_vacuum_gripper_finger" filename="libsticky_fingers.so">
         <capacity>1</capacity>
     </plugin>
     <contact>
-        <collision>[COLLISION NAME]</collision>
+        <collision>virtual_vacuum_gripper_collision</collision>
     </contact>
   </sensor>

Commit message: trying to add sticky fingers virtual vacuum gripper

File: Part_5/ur10_robot/ur10_launch/ur10_on_pedestal_w_sticky_fingers.xacro (robot description, xacro)
@@ -24,56 +24,10 @@
     <origin rpy="0 0 0 " xyz="0 0 0"/>
   </joint>
-  <link name= "virtual_vacuum_gripper">
-       <visual>
-      <geometry>
-         <cylinder length="0.02" radius="0.04"/>
-      </geometry>
-      <material name="blue">
-        <color rgba="0 0 .8 1"/>
-      </material>
-    </visual>
-    <collision name="virtual_vacuum_gripper_collision">
-      <origin rpy="0 0 0" xyz = "0 0 0"/>
-      <geometry>
-          <box size= "0.02 0.02 0.04"/>
-        <!--cylinder length="0.02" radius="0.04"/-->
-      </geometry>
-      <surface>
-          <friction>
-              <ode>
-                  <mu>30.0</mu>
-                  <mu2>30.0</mu2>
-              </ode>
-          </friction>
-          <contact>
-              <ode>
-                  <kp>100000.0</kp>
-                  <kd>100.0</kd>
-                  <max_vel>1.0</max_vel>
-                  <min_depth>0.001</min_depth>
-              </ode>
-          </contact>
-      </surface>
-    </collision>
-    <inertial>
-        <mass value = "0.05"/>
-        <inertia ixx = "0.01" iyy="0.01" izz="0.01" ixy="0.0" ixz="0.0" iyz="0.0" />
-    </inertial>
-  </link>
+  <xacro:include filename="$(find ur10_launch)/sticky_disc.urdf.xacro" />
   <joint name="gripper_joint" type="fixed">
     <parent link="tool0" />
     <!--ur10 base link is child-->
-    <child link="virtual_vacuum_gripper" />
-    <origin rpy="0 0 0 " xyz="0 0 0.0"/>
+    <child link="vvg" />
+    <origin rpy="0 0 0.01 " xyz="0 0 0.0"/>
   </joint>
-  <gazebo reference= "virtual_vacuum_gripper">
-  <sensor name="virtual_vacuum_gripper_sticky" type="contact">
-    <plugin name="virtual_vacuum_gripper_finger" filename="libsticky_fingers.so">
-        <capacity>1</capacity>
-    </plugin>
-    <contact>
-        <collision>virtual_vacuum_gripper_collision</collision>
-    </contact>
-  </sensor>
-</gazebo>
 </robot>

Commit message: got vacuum gripper working on UR10 other minor edits

File: Part_5/ur10_robot/ur10_launch/ur10_on_pedestal_w_sticky_fingers.xacro (robot description, xacro)
@@ -24,10 +24,38 @@
     <origin rpy="0 0 0 " xyz="0 0 0"/>
   </joint>
-  <xacro:include filename="$(find ur10_launch)/sticky_disc.urdf.xacro" />
+    <!--xacro:include filename="$(find ur10_launch)/sticky_disc.urdf.xacro" /-->
   <joint name="gripper_joint" type="fixed">
     <parent link="tool0" />
     <!--ur10 base link is child-->
     <child link="vvg" />
-    <origin rpy="0 0 0.01 " xyz="0 0 0.0"/>
+    <origin rpy="0 0 0" xyz="0 0 0.01"/>
+    <!---limit effort="0" velocity="0"/-->
   </joint>
+  <link name= "vvg">
+		<origin rpy="0 0 0 " xyz="0 0 0"/>
+		<visual>
+			<geometry>
+				<cylinder length="0.02" radius="0.04"/>
+			</geometry>
+			<material name="blue">
+				<color rgba="0 0 .8 1"/>
+			</material>
+		</visual>
+		<collision name="vvg_collision">
+			<geometry>
+              			<cylinder length="0.02" radius="0.04"/>
+			</geometry>
+		</collision>
+		<inertial>
+			<mass value="0.01"/>
+			<inertia ixx="1.0" ixy="0.0" ixz="0.0" iyy="1.0" iyz="0.0" izz="1.0"/>
+  		</inertial>
+	</link>
+  	<gazebo>
+		<plugin name="virtual_vacuum_gripper_finger" filename="libsticky_fingers.so">
+			<capacity>10</capacity>
+			<link>ur10_on_pedestal::wrist_3_link</link>
+			<!--link>ur10_on_pedestal::tool0</link-->
+		</plugin>
+	</gazebo>
 </robot>

Commit message: updates with ripple effects from manipulation abstraction

File: Part_5/ur10_robot/ur10_launch/ur10_on_pedestal_w_sticky_fingers.xacro (robot description, xacro)
@@ -6,7 +6,5 @@
     <xacro:arg name="gazebo" value="${gazebo}"/>
   </xacro:include>
-  <!--xacro:include filename="$(find baxter_description)/urdf/right_end_effector.urdf.xacro" /-->
-  <!--retrofit with Kinect and pedestal-->
-  <!--xacro:include filename="$(find baxter_variations)/kinect_link.urdf.xacro" /-->
+  <!--pedestal model-->
   <xacro:include filename="$(find ur10_launch)/ur10_pedestal.xacro" />
   <!-- attach robot base link to the pedestal -->
@@ -18,4 +16,5 @@
     <origin rpy="0 0 0 " xyz="0 0 0.426"/>
   </joint>
+  <!--attach the pedestal to the world-->
   <joint name="glue_base_to_world" type="fixed">
     <parent link="world" />
@@ -24,12 +23,5 @@
     <origin rpy="0 0 0 " xyz="0 0 0"/>
   </joint>
-    <!--xacro:include filename="$(find ur10_launch)/sticky_disc.urdf.xacro" /-->
-  <joint name="gripper_joint" type="fixed">
-    <parent link="tool0" />
-    <!--ur10 base link is child-->
-    <child link="vvg" />
-    <origin rpy="0 0 0" xyz="0 0 0.01"/>
-    <!---limit effort="0" velocity="0"/-->
-  </joint>
+  <!--define a link to emulate vacuum gripper-->
   <link name= "vvg">
 		<origin rpy="0 0 0 " xyz="0 0 0"/>
@@ -52,9 +44,15 @@
   		</inertial>
 	</link>
+  <!--attach virtual vacuum gripper, vvg, to tool flange-->
+  <joint name="gripper_joint" type="fixed">
+    <parent link="tool0" />
+    <child link="vvg" />
+    <origin rpy="0 0 0" xyz="0 0 0.01"/>
+  </joint>
+ <!-- bring in the sticky-fingers plug-in to simulate a vacuum gripper-->
   	<gazebo>
 		<plugin name="virtual_vacuum_gripper_finger" filename="libsticky_fingers.so">
 			<capacity>10</capacity>
 			<link>ur10_on_pedestal::wrist_3_link</link>
-			<!--link>ur10_on_pedestal::tool0</link-->
 		</plugin>
 	</gazebo>
