Commit message: changes for irb120 painting

File: Part_5/irb120/irb120_description/urdf/irb120.xacro (robot description, xacro)
@@ -20,4 +20,11 @@
     <child link="link1"/>
   </joint>
+  <!-- also, define a flange frame consistent w/ DH and IK library; z-axis pointing out from flange -->
+    <link name="flange_frame"/>
+  <joint name="flange_frame_jnt" type="fixed">
+    <parent link="link7"/>
+    <child link="flange_frame"/>
+    <origin xyz="0 0 0" rpy="0 1.5708 0"/>
+  </joint>
   <!-- Base Link -->
   <link name="link1">
@@ -252,5 +259,7 @@
     <type>transmission_interface/SimpleTransmission</type>
     <joint name="joint1">
-      <hardwareInterface>EffortJointInterface</hardwareInterface>
+      <hardwareInterface>EffortJointInterface</hardwareInterface>flange_stf
+[ INFO] [1512929221.358296873, 54.845000000]: frame_id: system_ref_frame
+[ INFO] [1512929221.358314256, 54.845000000]: child_frame_id: link7
     </joint>
     <actuator name="motor1">

Commit message: fixed collision model for irb120; more testing on cartesian planner

File: Part_5/irb120/irb120_description/urdf/irb120.xacro (robot description, xacro)
@@ -100,5 +100,5 @@
     <origin rpy="0 0 0" xyz="0 0 0.29"/>
     <axis xyz="0 1 0"/>
-    <limit effort="100" lower="-1.91986" upper="1.91986" velocity="4.36332"/>
+    <limit effort="500" lower="-1.91986" upper="1.91986" velocity="4.36332"/>
     <dynamics damping="1.7"/>
   </joint>
@@ -164,5 +164,6 @@
       <origin xyz="0 0 0" rpy="0 0 0"/>
       <geometry>
-	<box size="0.2 0.2 0.2"/>
+	<!--box size="${width} ${width} ${height3}"/-->
+	        <mesh filename="package://irb120_description/meshes/irb120/visual/link_4.stl"/>
       </geometry>
     </collision>
@@ -193,10 +194,10 @@
   </joint>
    <link name="link6">
-    <collision>
-      <origin xyz="0 0 0" rpy="0 0 0"/>
-      <geometry>
-	<box size="0.2 0.2 0.2"/>
-      </geometry>
-    </collision>
+    <!--collision>
+      <origin xyz="0 0 0" rpy="0 0 0"/>
+      <geometry>
+	        <mesh filename="package://irb120_description/meshes/irb120/visual/link_5.stl"/>
+      </geometry>
+    </collision-->
     <visual>
       <origin xyz="0 0 0" rpy="0 0 0"/>
@@ -226,7 +227,8 @@
    <link name="link7">
     <collision>
-      <origin xyz="0 0 0" rpy="0 0 0"/>
-      <geometry>
-	<box size="0.1 0.1 0.1"/>
+     <origin xyz="0 0 0" rpy="0 0 0"/>
+      <geometry>
+	<!--box size="${width} ${width} ${height3}"/-->
+	        <mesh filename="package://irb120_description/meshes/irb120/visual/link_6.stl"/>
       </geometry>
     </collision>

Commit message: lots of cartesian interface updates

File: Part_5/irb120/irb120_description/urdf/irb120.xacro (robot description, xacro)
@@ -105,10 +105,10 @@
   <!-- Top Link -->
   <link name="link3">
-    <collision>
+    <!--collision>
       <origin xyz="0 0 0" rpy="0 0 0"/>
       <geometry>
 	<box size="0.2 0.2 0.2"/>
       </geometry>
-    </collision>
+    </collision-->
     <visual>
       <origin xyz="0 0 0" rpy="0 0 0"/>
@@ -129,10 +129,10 @@
   </link>
   <link name="link4">
-    <collision>
+    <!--collision>
       <origin xyz="0 0 0" rpy="0 0 0"/>
       <geometry>
 	<box size="0.2 0.2 0.2"/>
       </geometry>
-    </collision>
+    </collision-->
     <visual>
       <origin xyz="0 0 0" rpy="0 0 0"/>
