Commit message: add code to launch Merrry/Jinx in Glennan 2nd floor

File: exmpl_models/glennan_2nd_flr/glennan_2nd_flr.urdf (robot description, URDF)
Before this commit: robot glennan_2nd_floor, 2 links, 1 joints
Links:
- link link: geometry collision mesh filename=package://exmpl_models/glennan_2nd_flr/glennan_2nd_flr.stl; visual mesh filename=package://exmpl_models/glennan_2nd_flr/glennan_2nd_flr.stl
